File: MyAIQuadrapedRobot_HW/1000027_V0/1000027_V0.kicad_pcb (KiCad board)
At the start: 2 copper layers, 40.1 x 43.8 mm, 4 parts, among them J1 MTSW-106-12-L-S-790_6_by_1_he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, J2 10076801-406T18LF_9_by_2_head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, J3 533750410, J4 0525591853

Commit message: KiCad library update complete.
Parts:
- J1: value MTSW-106-12-L-S-790_6_by_1_header -> 10076801-406T18LF_9_by_2_header; footprint CatBot_JSC:SAMTEC_MTSW-106-12-L-S-790 -> myKiCadGlobalFootprintLibrary:AMPHENOL_10076801-406T18LF
- J2: value 10076801-406T18LF_9_by_2_header -> 0525591853; footprint CatBot_JSC:AMPHENOL_10076801-406T18LF -> myKiCadGlobalFootprintLibrary:525591853
- J3: value 533750410 -> MTSW-106-12-L-S-790_6_by_1_header; footprint Molex_connectors_JSC:MOLEX_533750410 -> myKiCadGlobalFootprintLibrary:SAMTEC_MTSW-106-12-L-S-790
- J4: value 0525591853 -> MOLEX_533750410; footprint Molex_connectors_JSC:CON_525591853_MOL -> myKiCadGlobalFootprintLibrary:533750410
- moved J4 22.3 mm to (169.2, 75.9)
- moved J1 18.3 mm to (165.6, 64.6), turned to 180 degrees
- moved J2 10.9 mm to (165.9, 52.5), turned to 0 degrees
- moved J3 7.82 mm to (165.4, 82.6)
Connections:
- J1 pad 01: /GND -> C1
- J1 pad 02: unconnected-(J1-Pad02) -> C2
- J1 pad 03: /SCL -> C3
- J1 pad 04: /SDA -> C4
- J1 pad 05: /Vcc (3.3V) -> C5
- J1 pad 06: unconnected-(J1-Pad06) -> C6
- J4 pad 1: C1 -> /GND
- J4 pad 2: C2 -> /SCL
- J4 pad 3: C3 -> /SDA
- J4 pad 4: C4 -> /Vcc (3.3V)
Routing:
- net C18: track 15.2 -> 0.00 mm
- net C16: track 12.9 -> 0.00 mm
- net C14: track 12.1 -> 0.00 mm
- net C15: track 12.0 -> 0.00 mm
- net C2: track 11.7 -> 0.00 mm
- net C17: track 11.7 -> 0.00 mm
- net C1: track 11.6 -> 0.00 mm, vias 1 -> 0
- net C4: track 11.1 -> 0.00 mm
- net C3: track 10.9 -> 0.00 mm, vias 1 -> 0
- net C12: track 10.5 -> 0.00 mm
- net C13: track 10.4 -> 0.00 mm
- net C6: track 10.4 -> 0.00 mm
- net C5: track 10.2 -> 0.00 mm, vias 1 -> 0
- net C10: track 9.84 -> 0.00 mm
- net C8: track 9.77 -> 0.00 mm
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
Commit message: 1000027_V0(a) ready for checking.
Parts:
- J4: value MOLEX_533750410 -> 533750410
- moved J3 28.6 mm to (149.5, 106.3)
- moved J1 28.5 mm to (149.4, 88.0)
- moved J2 28.5 mm to (149.3, 75.6)
- moved J4 28.1 mm to (153.4, 99.1)
Routing:
- net C17: track 0.00 -> 17.3 mm, vias 0 -> 1
- net C16: track 0.00 -> 17.1 mm
- net C18: track 0.00 -> 16.8 mm
- net C14: track 0.00 -> 15.8 mm
- net C15: track 0.00 -> 15.2 mm, vias 0 -> 1
- net C2: track 0.00 -> 14.7 mm
- net C1: track 0.00 -> 14.2 mm, vias 0 -> 1
- net C13: track 0.00 -> 14.2 mm, vias 0 -> 1
- net C12: track 0.00 -> 14.2 mm
- net C4: track 0.00 -> 14.0 mm
- net C3: track 0.00 -> 13.6 mm, vias 0 -> 1
- net C6: track 0.00 -> 13.5 mm
- net C5: track 0.00 -> 13.2 mm, vias 0 -> 1
- net C11: track 0.00 -> 13.1 mm, vias 0 -> 1
- net C10: track 0.00 -> 13.1 mm
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Other:
- outline, holes or cut-outs redrawn
- board text added: "1000027_V0a 1 of 2 Copyright © James Canova, June 2023, Victoria, BC Canada"
- board text added: "1000027_V0a 2 of 2 Copyright © James Canova, June 2023, Victoria, BC Canada"
- board text added: "↑ IN"
- board text added: "↑ UP"
