File: MyAIQuadrapedRobot_HW/1000027_V0/1000027_V0.kicad_sch (KiCad schematic)
At the start: 4 parts, among them J1 MTSW-106-12-L-S-790_6_by_1_he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, J2 10076801-406T18LF_9_by_2_head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, J3 533750410, J4 0525591853

Commit message: KiCad library update complete.
Parts:
- J1: renamed from J2; footprint AMPHENOL_10076801-406T18LF -> myKiCadGlobalFootprintLibrary:AMPHENOL_10076801-406T18LF; symbol CatBot_JSC:10076801-406T18LF_9_by_2_header -> myKiCadGlobalSymbolLibrary:10076801-406T18LF
- J2: renamed from J4; footprint Molex_connectors_JSC:CON_525591853_MOL -> myKiCadGlobalFootprintLibrary:525591853; symbol Molex_connectors_JSC:0525591853 -> myKiCadGlobalSymbolLibrary:525591853
- J3: renamed from J1; symbol CatBot_JSC:MTSW-106-12-L-S-790_6_by_1_header -> myKiCadGlobalSymbolLibrary:MTSW-106-12-L-S-790
- J4: renamed from J3; footprint Molex_connectors_JSC:MOLEX_533750410 -> myKiCadGlobalFootprintLibrary:533750410; symbol Molex_connectors_JSC:533750410 -> myKiCadGlobalSymbolLibrary:533750410
Changed lines of the file:
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@@
     (effects (font (size 1.27 1.27)) (justify left bottom))
   )
-  (text "Connector on camera." (at 58.42 45.212 0)
+  (text "Connector on camera." (at 64.008 41.91 0)
     (effects (font (size 1.27 1.27)) (justify left bottom))
   )
@@
     )
   )
-  (symbol (lib_id "CatBot_JSC:10076801-406T18LF_9_by_2_header") (at 110.236 99.822 270) (mirror x) (unit 1)
+  (symbol (lib_id "myKiCadGlobalSymbolLibrary:10076801-406T18LF") (at 110.236 99.822 270) (mirror x) (unit 1)
     (in_bom yes) (on_board yes) (fields_autoplaced)
-    (property "Reference" "J2" (id 0) (at 124.714 99.8219 90)
+    (property "Reference" "J1" (id 0) (at 124.46 99.8219 90)
       (effects (font (size 1.27 1.27)) (justify left))
     )
@@
       (effects (font (size 1.27 1.27)) (justify left) hide)
     )
-    (property "Footprint" "AMPHENOL_10076801-406T18LF" (id 2) (at 87.376 99.568 0)
+    (property "Footprint" "myKiCadGlobalFootprintLibrary:AMPHENOL_10076801-406T18LF" (id 2) (at 89.154 99.568 0)
       (effects (font (size 1.27 1.27)) (justify bottom) hide)
     )
@@
       (effects (font (size 1.27 1.27)) (justify bottom) hide)
     )
-    (property "MANUFACTURER" "Amphenol ICC (FCI)" (id 5) (at 83.82 100.076 0)
-      (effects (font (size 1.27 1.27)) (justify bottom) hide)
-    )
-    (property "STANDARD" "Manufacturer Recommendations" (id 6) (at 89.916 99.06 0)
+    (property "MANUFACTURER" "Amphenol ICC (FCI)" (id 5) (at 93.472 98.298 0)
+      (effects (font (size 1.27 1.27)) (justify bottom) hide)
+    )
+    (property "STANDARD" "Manufacturer Recommendations" (id 6) (at 91.44 100.076 0)
       (effects (font (size 1.27 1.27)) (justify bottom) hide)
     )
@@
     (pin "18")
   )
-  (symbol (lib_id "CatBot_JSC:MTSW-106-12-L-S-790_6_by_1_header") (at 210.058 86.868 270) (unit 1)
+  (symbol (lib_id "myKiCadGlobalSymbolLibrary:MTSW-106-12-L-S-790") (at 210.058 86.868 270) (unit 1)
     (in_bom yes) (on_board yes) (fields_autoplaced)
-    (property "Reference" "J1" (id 0) (at 220.98 86.8679 90)
+    (property "Reference" "J3" (id 0) (at 220.98 86.8679 90)
       (effects (font (size 1.27 1.27)) (justify left))
     )
@@
       (effects (font (size 1.27 1.27)) (justify left) hide)
     )
-    (property "Footprint" "SAMTEC_MTSW-106-12-L-S-790" (id 2) (at 188.214 85.598 0)
+    (property "Footprint" "SAMTEC_MTSW-106-12-L-S-790" (id 2) (at 194.056 87.884 0)
       (effects (font (size 1.27 1.27)) (justify bottom) hide)
     )
@@
       (effects (font (size 1.27 1.27)) (justify bottom) hide)
     )
-    (property "MANUFACTURER" "Samtec" (id 5) (at 191.008 85.598 0)
-      (effects (font (size 1.27 1.27)) (justify bottom) hide)
-    )
-    (property "STANDARD" "Manufacturer Recommendations" (id 6) (at 193.802 85.344 0)
+    (property "MANUFACTURER" "Samtec" (id 5) (at 197.104 86.36 0)
+      (effects (font (size 1.27 1.27)) (justify bottom) hide)
+    )
+    (property "STANDARD" "Manufacturer Recommendations" (id 6) (at 225.806 86.106 0)
       (effects (font (size 1.27 1.27)) (justify bottom) hide)
     )
@@
     (pin "06")
   )
-  (symbol (lib_id "Molex_connectors_JSC:533750410") (at 212.09 61.722 270) (mirror x) (unit 1)
+  (symbol (lib_id "myKiCadGlobalSymbolLibrary:533750410") (at 212.09 61.722 270) (mirror x) (unit 1)
     (in_bom yes) (on_board yes) (fields_autoplaced)
-    (property "Reference" "J3" (id 0) (at 218.186 57.9119 90)
+    (property "Reference" "J4" (id 0) (at 218.44 57.9119 90)
       (effects (font (size 1.27 1.27)) (justify left))
     )
@@
       (effects (font (size 1.27 1.27)) (justify left) hide)
     )
-    (property "Footprint" "Molex_connectors_JSC:MOLEX_533750410" (id 2) (at 218.186 60.4519 90)
-      (effects (font (size 1.27 1.27)) (justify left) hide)
+    (property "Footprint" "myKiCadGlobalFootprintLibrary:533750410" (id 2) (at 184.658 60.198 0)
+      (effects (font (size 1.27 1.27)) (justify bottom) hide)
     )
     (property "Datasheet" "" (id 3) (at 212.09 61.722 0)
       (effects (font (size 1.27 1.27)) hide)
     )
-    (property "PARTREV" "C" (id 4) (at 212.09 61.722 0)
-      (effects (font (size 1.27 1.27)) (justify bottom) hide)
-    )
-    (property "STANDARD" "Manufacturer Recommendations" (id 5) (at 199.39 62.23 0)
-      (effects (font (size 1.27 1.27)) (justify bottom) hide)
-    )
-    (property "MAXIMUM_PACKAGE_HEIGHT" "11.75 mm" (id 6) (at 197.612 61.214 0)
-      (effects (font (size 1.27 1.27)) (justify bottom) hide)
-    )
-    (property "MANUFACTURER" "Molex" (id 7) (at 197.358 45.466 0)
+    (property "PARTREV" "C" (id 4) (at 187.198 48.768 0)
+      (effects (font (size 1.27 1.27)) (justify bottom) hide)
+    )
+    (property "STANDARD" "Manufacturer Recommendations" (id 5) (at 193.548 57.404 0)
+      (effects (font (size 1.27 1.27)) (justify bottom) hide)
+    )
+    (property "MAXIMUM_PACKAGE_HEIGHT" "11.75 mm" (id 6) (at 189.738 58.928 0)
+      (effects (font (size 1.27 1.27)) (justify bottom) hide)
+    )
+    (property "MANUFACTURER" "Molex" (id 7) (at 186.69 73.152 0)
       (effects (font (size 1.27 1.27)) (justify bottom) hide)
     )
@@
     (pin "4")
   )
-  (symbol (lib_id "Molex_connectors_JSC:0525591853") (at 133.35 48.768 270) (mirror x) (unit 1)
+  (symbol (lib_id "myKiCadGlobalSymbolLibrary:525591853") (at 133.35 48.768 270) (mirror x) (unit 1)
     (in_bom yes) (on_board yes)
-    (property "Reference" "J4" (id 0) (at 138.43 39.878 90)
+    (property "Reference" "J2" (id 0) (at 138.43 39.878 90)
       (effects (font (size 1.524 1.524)))
     )
@@
       (effects (font (size 1.524 1.524)) hide)
     )
-    (property "Footprint" "Molex_connectors_JSC:CON_525591853_MOL" (id 2) (at 111.887 33.274 90)
+    (property "Footprint" "myKiCadGlobalFootprintLibrary:525591853" (id 2) (at 108.0771 35.052 0)
+      (effects (font (size 1.27 1.27) italic) (justify left) hide)
+    )
+    (property "Datasheet" "559171630" (id 3) (at 133.35 48.768 0)
       (effects (font (size 1.27 1.27) italic) hide)
     )
-    (property "Datasheet" "559171630" (id 3) (at 130.302 27.432 0)
-      (effects (font (size 1.27 1.27) italic) hide)
+    (property "Field4" "" (id 4) (at 133.35 48.768 0)
+      (effects (font (size 1.27 1.27)) hide)
     )
     (pin "1")
@@
   )
   (symbol_instances
+    (path "/73d8daea-e7b8-4724-99fc-3fc975463057"
+      (reference "J1") (unit 1) (value "10076801-406T18LF_9_by_2_header") (footprint "myKiCadGlobalFootprintLibrary:AMPHENOL_10076801-406T18LF")
+    )
+    (path "/d984850c-7f3e-4675-94fa-167484fc996d"
+      (reference "J2") (unit 1) (value "0525591853") (footprint "myKiCadGlobalFootprintLibrary:525591853")
+    )
     (path "/a98fe8de-3542-4db9-a3d5-cada9dd22f37"
-      (reference "J1") (unit 1) (value "MTSW-106-12-L-S-790_6_by_1_header") (footprint "SAMTEC_MTSW-106-12-L-S-790")
-    )
-    (path "/73d8daea-e7b8-4724-99fc-3fc975463057"
-      (reference "J2") (unit 1) (value "10076801-406T18LF_9_by_2_header") (footprint "AMPHENOL_10076801-406T18LF")
+      (reference "J3") (unit 1) (value "MTSW-106-12-L-S-790_6_by_1_header") (footprint "SAMTEC_MTSW-106-12-L-S-790")
     )
     (path "/c7606c1a-033f-4927-8400-7499dfa20240"
-      (reference "J3") (unit 1) (value "533750410") (footprint "Molex_connectors_JSC:MOLEX_533750410")
-    )
-    (path "/d984850c-7f3e-4675-94fa-167484fc996d"
-      (reference "J4") (unit 1) (value "0525591853") (footprint "Molex_connectors_JSC:CON_525591853_MOL")
-    )
-  )
+      (reference "J4") (unit 1) (value "533750410") (footprint "myKiCadGlobalFootprintLibrary:533750410")
+    )
+  )

Commit message: Start of version V0b.
Other:
- note removed: "Connector on camera."
- note removed: "Connector on main PCB."
Changed lines of the file:
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@@
     (stroke (width 0) (type default) (color 0 0 0 0))
-  )
-  (text "Connector on \nmain PCB." (at 71.374 103.886 0)
-    (effects (font (size 1.27 1.27)) (justify left bottom))
-  )
-  (text "Connector on camera." (at 64.008 41.91 0)
-    (effects (font (size 1.27 1.27)) (justify left bottom))
   )
   (label "GND" (at 216.154 69.342 0)
