File: MyAIQuadrapedRobot_HW/1000026_V0/1000026_V0.kicad_pcb.kicad_sch (KiCad schematic)
At the start: 27 parts, among them J2 0525591853, J3 532580229, J5 532580229, J7 533750410, J9 0525591853, SW1 TL3305CF260QG, U1 TXB0108PWR, U2 MAX7480ESA+

Commit message: Development changes.
Parts:
- A1, A2: footprint CatBot_JSC:Arduino_BLE_33 -> myKiCadGlobalFootprintLibrary:Nano33BLE_with_headers; symbol CatBot_JSC:Arduino_BLE_33 -> myKiCadGlobalSymbolLibrary:Arduino_BLE_33
- H1, H2, H3, H4: footprint MountingHole:MountingHole_2.2mm_M2 -> myKiCadGlobalFootprintLibrary:MountingHole_2.2mm_M2; symbol Mechanical:MountingHole -> myKiCadGlobalSymbolLibrary:MountingHole
- R1: footprint CatBot_JSC:300_Ohm_RESC6332X70N -> myKiCadGlobalFootprintLibrary:RESC6332X70N; symbol CatBot_JSC:RMCF2512FT330R -> myKiCadGlobalSymbolLibrary:RMCF2512FT330R; Resistance (none) -> 300 Ω
- SW1: footprint CatBot_JSC:Push_Button_Switch_SW4_TL3305CF260QG_EWI-M -> myKiCadGlobalFootprintLibrary:TL3305CF260QG; symbol CatBot_JSC:TL3305CF260QG -> myKiCadGlobalSymbolLibrary:TL3305CF260QG
Connections:
- net 7.4V: now also R1.1; no longer R1.2
- net at LED1.2: now also R1.2; no longer R1.1
Changed lines of the file:
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@@
+    (stroke (width 0) (type default) (color 0 0 0 0))
+  )
+  (wire (pts (xy 92.71 148.082) (xy 92.71 147.32))
     (stroke (width 0) (type default) (color 0 0 0 0))
   )
@@
     (pin "2")
   )
-  (symbol (lib_id "Mechanical:MountingHole") (at 153.162 182.372 0) (unit 1)
+  (symbol (lib_id "myKiCadGlobalSymbolLibrary:MountingHole") (at 153.162 182.372 0) (unit 1)
     (in_bom yes) (on_board yes)
     (property "Reference" "H4" (id 0) (at 155.956 181.1019 0)
@@
       (effects (font (size 1.27 1.27)) (justify left))
     )
-    (property "Footprint" "MountingHole:MountingHole_2.2mm_M2" (id 2) (at 153.416 178.562 0)
+    (property "Footprint" "myKiCadGlobalFootprintLibrary:MountingHole_2.2mm_M2" (id 2) (at 153.162 182.372 0)
       (effects (font (size 1.27 1.27)) hide)
     )
@@
     )
   )
-  (symbol (lib_id "CatBot_JSC:Arduino_BLE_33") (at 203.2 53.34 180) (unit 1)
+  (symbol (lib_id "myKiCadGlobalSymbolLibrary:Arduino_BLE_33") (at 203.2 53.34 180) (unit 1)
     (in_bom yes) (on_board yes)
     (property "Reference" "A1" (id 0) (at 203.2 27.686 0))
     (property "Value" "Arduino_Nano_BLE_33_SENSE" (id 1) (at 203.2 29.718 0))
-    (property "Footprint" "CatBot_JSC:Arduino_BLE_33" (id 2) (at 217.17 83.82 0)
-      (effects (font (size 1.27 1.27) italic) hide)
-    )
-    (property "Datasheet" "https://www.arduino.cc/en/uploads/Main/ArduinoNanoManual23.pdf.TBD" (id 3) (at 196.85 19.05 0)
+    (property "Footprint" "myKiCadGlobalFootprintLibrary:Nano33BLE_with_headers" (id 2) (at 189.23 22.86 0)
+      (effects (font (size 1.27 1.27) italic))
+    )
+    (property "Datasheet" "https://www.arduino.cc/en/uploads/Main/ArduinoNanoManual23.pdf.TBD" (id 3) (at 209.55 87.63 0)
       (effects (font (size 1.27 1.27)) hide)
     )
@@
     (pin "2")
   )
-  (symbol (lib_id "Mechanical:MountingHole") (at 153.162 176.784 0) (unit 1)
+  (symbol (lib_id "myKiCadGlobalSymbolLibrary:MountingHole") (at 153.162 176.784 0) (unit 1)
     (in_bom yes) (on_board yes)
     (property "Reference" "H3" (id 0) (at 155.956 175.5139 0)
@@
       (effects (font (size 1.27 1.27)) (justify left))
     )
-    (property "Footprint" "MountingHole:MountingHole_2.2mm_M2" (id 2) (at 153.416 172.974 0)
+    (property "Footprint" "myKiCadGlobalFootprintLibrary:MountingHole_2.2mm_M2" (id 2) (at 153.162 176.784 0)
       (effects (font (size 1.27 1.27)) hide)
     )
@@
     (pin "2")
   )
-  (symbol (lib_id "CatBot_JSC:RMCF2512FT330R") (at 92.202 138.176 90) (unit 1)
-    (in_bom yes) (on_board yes)
-    (property "Reference" "R1" (id 0) (at 89.916 137.922 0))
-    (property "Value" "RMCF2512FT330R" (id 1) (at 98.806 139.954 0)
-      (effects (font (size 1.27 1.27)) hide)
-    )
-    (property "Footprint" "CatBot_JSC:300_Ohm_RESC6332X70N" (id 2) (at 88.138 139.7 0)
-      (effects (font (size 1.27 1.27)) hide)
-    )
-    (property "Datasheet" "" (id 3) (at 92.202 138.176 0)
-      (effects (font (size 1.27 1.27)) hide)
-    )
+  (symbol (lib_id "myKiCadGlobalSymbolLibrary:RMCF2512FT330R") (at 92.71 138.938 90) (unit 1)
+    (in_bom yes) (on_board yes)
+    (property "Reference" "R1" (id 0) (at 96.266 137.668 0))
+    (property "Value" "RMCF2512FT330R" (id 1) (at 86.106 137.16 0)
+      (effects (font (size 1.27 1.27)) hide)
+    )
+    (property "Footprint" "myKiCadGlobalFootprintLibrary:RESC6332X70N" (id 2) (at 101.854 140.462 0)
+      (effects (font (size 1.27 1.27)) (justify bottom) hide)
+    )
+    (property "Datasheet" "" (id 3) (at 92.71 138.938 0)
+      (effects (font (size 1.27 1.27)) hide)
+    )
+    (property "Resistance" "300 Ω" (id 4) (at 89.408 137.668 0))
     (pin "1")
     (pin "2")
@@
     (pin "2")
   )
-  (symbol (lib_id "CatBot_JSC:TL3305CF260QG") (at 180.594 96.52 0) (unit 1)
+  (symbol (lib_id "myKiCadGlobalSymbolLibrary:TL3305CF260QG") (at 180.594 96.52 0) (unit 1)
     (in_bom yes) (on_board yes) (fields_autoplaced)
     (property "Reference" "SW1" (id 0) (at 200.914 89.408 0)
@@
       (effects (font (size 1.524 1.524)) hide)
     )
-    (property "Footprint" "CatBot_JSC:Push_Button_Switch_SW4_TL3305CF260QG_EWI-M" (id 2) (at 165.735 101.346 0)
-      (effects (font (size 1.27 1.27) italic) hide)
-    )
-    (property "Datasheet" "TL3305CF260QG" (id 3) (at 180.594 96.52 0)
+    (property "Footprint" "myKiCadGlobalFootprintLibrary:TL3305CF260QG" (id 2) (at 203.708 112.014 0)
+      (effects (font (size 1.27 1.27) italic) hide)
+    )
+    (property "Datasheet" "TL3305CF260QG" (id 3) (at 201.676 108.204 0)
       (effects (font (size 1.27 1.27) italic) hide)
     )
@@
     (pin "9")
   )
-  (symbol (lib_id "Mechanical:MountingHole") (at 131.826 182.372 0) (unit 1)
+  (symbol (lib_id "myKiCadGlobalSymbolLibrary:MountingHole") (at 131.826 182.372 0) (unit 1)
     (in_bom yes) (on_board yes)
     (property "Reference" "H2" (id 0) (at 134.62 181.1019 0)
@@
       (effects (font (size 1.27 1.27)) (justify left))
     )
-    (property "Footprint" "MountingHole:MountingHole_2.2mm_M2" (id 2) (at 132.08 178.562 0)
+    (property "Footprint" "myKiCadGlobalFootprintLibrary:MountingHole_2.2mm_M2" (id 2) (at 131.826 182.372 0)
       (effects (font (size 1.27 1.27)) hide)
     )
@@
     )
   )
-  (symbol (lib_id "Power_library:GNDREF") (at 232.918 159.512 0) (unit 1)
+  (symbol (lib_id "myKiCadGlobalSymbolLibrary:GNDREF") (at 232.918 159.512 0) (unit 1)
     (in_bom yes) (on_board yes)
     (property "Reference" "#PWR0103" (id 0) (at 232.918 165.862 0)
@@
     (pin "2")
   )
-  (symbol (lib_id "Power_library:GNDREF") (at 41.148 171.704 0) (unit 1)
+  (symbol (lib_id "myKiCadGlobalSymbolLibrary:GNDREF") (at 41.148 171.704 0) (unit 1)
     (in_bom yes) (on_board yes)
     (property "Reference" "#PWR0102" (id 0) (at 41.148 178.054 0)
@@
     (pin "1")
   )
-  (symbol (lib_id "Mechanical:MountingHole") (at 131.826 176.784 0) (unit 1)
+  (symbol (lib_id "myKiCadGlobalSymbolLibrary:MountingHole") (at 131.826 176.784 0) (unit 1)
     (in_bom yes) (on_board yes)
     (property "Reference" "H1" (id 0) (at 134.62 175.5139 0)
@@
       (effects (font (size 1.27 1.27)) (justify left))
     )
-    (property "Footprint" "MountingHole:MountingHole_2.2mm_M2" (id 2) (at 132.08 172.974 0)
+    (property "Footprint" "myKiCadGlobalFootprintLibrary:MountingHole_2.2mm_M2" (id 2) (at 131.826 176.784 0)
       (effects (font (size 1.27 1.27)) hide)
     )
@@
     (pin "2")
   )
-  (symbol (lib_id "CatBot_JSC:Arduino_BLE_33") (at 137.414 52.324 180) (unit 1)
+  (symbol (lib_id "myKiCadGlobalSymbolLibrary:Arduino_BLE_33") (at 137.414 52.324 180) (unit 1)
     (in_bom yes) (on_board yes) (fields_autoplaced)
     (property "Reference" "A2" (id 0) (at 137.414 25.654 0))
     (property "Value" "Arduino_Nano_BLE_33" (id 1) (at 137.414 28.194 0))
-    (property "Footprint" "CatBot_JSC:Arduino_BLE_33" (id 2) (at 151.384 82.804 0)
-      (effects (font (size 1.27 1.27) italic) hide)
-    )
-    (property "Datasheet" "https://www.arduino.cc/en/uploads/Main/ArduinoNanoManual23.pdf.TBD" (id 3) (at 131.064 18.034 0)
+    (property "Footprint" "myKiCadGlobalFootprintLibrary:Nano33BLE_with_headers" (id 2) (at 123.444 21.844 0)
+      (effects (font (size 1.27 1.27) italic))
+    )
+    (property "Datasheet" "https://www.arduino.cc/en/uploads/Main/ArduinoNanoManual23.pdf.TBD" (id 3) (at 143.764 86.614 0)
       (effects (font (size 1.27 1.27)) hide)
     )
@@
     )
     (path "/153f53fc-5f44-4cd5-9329-7b7a52a06b3c"
-      (reference "A1") (unit 1) (value "Arduino_Nano_BLE_33_SENSE") (footprint "CatBot_JSC:Arduino_BLE_33")
+      (reference "A1") (unit 1) (value "Arduino_Nano_BLE_33_SENSE") (footprint "myKiCadGlobalFootprintLibrary:Nano33BLE_with_headers")
     )
     (path "/fe77efe3-e56e-4eb7-b9b3-8508e79243c3"
-      (reference "A2") (unit 1) (value "Arduino_Nano_BLE_33") (footprint "CatBot_JSC:Arduino_BLE_33")
+      (reference "A2") (unit 1) (value "Arduino_Nano_BLE_33") (footprint "myKiCadGlobalFootprintLibrary:Nano33BLE_with_headers")
     )
     (path "/c5733604-1d59-4eef-a155-77e6e603be57"
@@
     )
     (path "/ef59e5db-1a94-4e40-bec0-10bb11caf784"
-      (reference "H1") (unit 1) (value "MountingHole") (footprint "MountingHole:MountingHole_2.2mm_M2")
+      (reference "H1") (unit 1) (value "MountingHole") (footprint "myKiCadGlobalFootprintLibrary:MountingHole_2.2mm_M2")
     )
     (path "/b08ea753-8db4-46e2-b3e2-f49619fafa59"
-      (reference "H2") (unit 1) (value "MountingHole") (footprint "MountingHole:MountingHole_2.2mm_M2")
+      (reference "H2") (unit 1) (value "MountingHole") (footprint "myKiCadGlobalFootprintLibrary:MountingHole_2.2mm_M2")
     )
     (path "/2828fb95-f19a-4bfa-acd3-37866c09b606"
-      (reference "H3") (unit 1) (value "MountingHole") (footprint "MountingHole:MountingHole_2.2mm_M2")
+      (reference "H3") (unit 1) (value "MountingHole") (footprint "myKiCadGlobalFootprintLibrary:MountingHole_2.2mm_M2")
     )
     (path "/108c5b5e-7876-4972-9fb9-47a0ce63bdba"
-      (reference "H4") (unit 1) (value "MountingHole") (footprint "MountingHole:MountingHole_2.2mm_M2")
+      (reference "H4") (unit 1) (value "MountingHole") (footprint "myKiCadGlobalFootprintLibrary:MountingHole_2.2mm_M2")
     )
     (path "/7449cb12-a7dc-45a3-9f86-ab09afa5da9d"
@@
     )
     (path "/313c8f60-e002-4e09-936b-cb34afac17da"
-      (reference "R1") (unit 1) (value "RMCF2512FT330R") (footprint "CatBot_JSC:300_Ohm_RESC6332X70N")
+      (reference "R1") (unit 1) (value "RMCF2512FT330R") (footprint "myKiCadGlobalFootprintLibrary:RESC6332X70N")
     )
     (path "/08e3cfd4-04f7-4705-867c-0422902dcf75"
@@
     )
     (path "/57dff52c-52c3-44d4-87a2-0d4b53b1b943"
-      (reference "SW1") (unit 1) (value "TL3305CF260QG") (footprint "CatBot_JSC:Push_Button_Switch_SW4_TL3305CF260QG_EWI-M")
+      (reference "SW1") (unit 1) (value "TL3305CF260QG") (footprint "myKiCadGlobalFootprintLibrary:TL3305CF260QG")
     )
     (path "/6d2a8fd8-9cd6-41ea-805c-4a71d7617c50"

Commit message: Update of KiCad library in progress.
Parts:
- removed C2, C3, C5, C6: CL05A104KA5NNNC_0pt1uF, CatBot_JSC:CAPC1005X55N, symbol CatBot_JSC:CL05A104KA5NNNC_0pt1uF
- added C2, C3, C4, C5: CL05A104KA5NNNC, myKiCadGlobalFootprintLibrary:CAPC1005X55N, symbol myKiCadGlobalSymbolLibrary:CL05A104KA5NNNC
- C1: value CL05A104KA5NNNC_0pt1uF -> 12065C503JAT2A; footprint CatBot_JSC:CAPC1005X55N -> myKiCadGlobalFootprintLibrary:12065C503JAT2A; symbol CatBot_JSC:CL05A104KA5NNNC_0pt1uF -> myKiCadGlobalSymbolLibrary:12065C503JAT2A; Capacitance (none) -> 0.05uF; Note 0.1uF -> (none)
- D1, D2, D3: footprint CatBot_JSC:Diode_CR_SOD323_MCC-M -> myKiCadGlobalFootprintLibrary:1N4148WT; symbol CatBot_JSC:1N4148WX-TP -> myKiCadGlobalSymbolLibrary:1N4148WX-TP
- F1: footprint CatBot_JSC:RGEF300 -> myKiCadGlobalFootprintLibrary:RGEF300HF
- J3, J5: footprint Molex_connectors_JSC:CON_532580229_MOL -> myKiCadGlobalFootprintLibrary:0532580229; symbol Molex_connectors_JSC:532580229 -> myKiCadGlobalSymbolLibrary:532580229
- LED1: footprint CatBot_JSC:Led_green_C503B -> myKiCadGlobalFootprintLibrary:C503B-GAN-CB0F0791; symbol CatBot_JSC:C503B-GAN-CB0F0791 -> myKiCadGlobalSymbolLibrary:C503B-GAN-CB0F0791
- R2: footprint CatBot_JSC:RC0402JR-0710KL -> myKiCadGlobalFootprintLibrary:RC0402JR-0710KL; symbol CatBot_JSC:RC0402JR-0710KL -> myKiCadGlobalSymbolLibrary:RC0402JR-0710KL
- S1: footprint CatBot_JSC:Slider_switch_500SSP1S2M2QEA -> myKiCadGlobalFootprintLibrary:500SSP1S2M2QEA
- U2: footprint CatBot_JSC:SOIC127P600X175-8N_MAX7480 -> myKiCadGlobalFootprintLibrary:MAX7480ESA; symbol CatBot_JSC:MAX7480ESA+ -> myKiCadGlobalSymbolLibrary:MAX7480ESA+
Connections:
- net 3.3V_2: now also C3.1
- net 5V_1: now also C4.1; no longer U2.4 (VDD)
- net 5V_2: now also C2.1
- net CLK: now also C1.2; no longer C1.1
- net COM: now also C5.1
- net GNDREF: now also C1.1, U2.4 (VDD), C2.2, C3.2, C4.2, C5.2; no longer C1.2
Other:
- moved on the sheet: D2

Commit message: KiCad library update complete.
Parts:
- F1: symbol CatBot_JSC:RGEF300_Fuse -> myKiCadGlobalSymbolLibrary:FUSE
- J1: renamed from J7; footprint Molex_connectors_JSC:MOLEX_533750410 -> myKiCadGlobalFootprintLibrary:533750410; symbol Molex_connectors_JSC:533750410 -> myKiCadGlobalSymbolLibrary:533750410
- J2, J9: footprint Molex_connectors_JSC:CON_525591853_MOL -> myKiCadGlobalFootprintLibrary:525591853; symbol Molex_connectors_JSC:0525591853 -> myKiCadGlobalSymbolLibrary:525591853
- S1: symbol CatBot_JSC:500SSP1S2M2QEA -> myKiCadGlobalSymbolLibrary:500SSP1S2M2QEA
Changed lines of the file:
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@@
     (pin "2")
   )
-  (symbol (lib_id "CatBot_JSC:500SSP1S2M2QEA") (at 70.866 149.86 0) (unit 1)
+  (symbol (lib_id "myKiCadGlobalSymbolLibrary:500SSP1S2M2QEA") (at 70.866 149.86 0) (unit 1)
     (in_bom yes) (on_board yes) (fields_autoplaced)
     (property "Reference" "S1" (id 0) (at 70.866 144.272 0))
@@
       (effects (font (size 1.27 1.27)) hide)
     )
-    (property "Footprint" "myKiCadGlobalFootprintLibrary:500SSP1S2M2QEA" (id 2) (at 71.9074 145.9992 0)
+    (property "Footprint" "myKiCadGlobalFootprintLibrary:500SSP1S2M2QEA" (id 2) (at 73.152 166.624 0)
       (effects (font (size 1.27 1.27)) (justify bottom) hide)
     )
@@
       (effects (font (size 1.27 1.27)) hide)
     )
-    (property "PARTREV" "C" (id 4) (at 70.866 149.86 0)
-      (effects (font (size 1.27 1.27)) (justify bottom) hide)
-    )
-    (property "STANDARD" "Manufacturer Recommendations" (id 5) (at 70.6374 142.2654 0)
-      (effects (font (size 1.27 1.27)) (justify bottom) hide)
-    )
-    (property "MAXIMUM_PACKAGE_HEIGHT" "13.59mm" (id 6) (at 66.0654 159.258 0)
-      (effects (font (size 1.27 1.27)) (justify bottom) hide)
-    )
-    (property "MANUFACTURER" "E-switch" (id 7) (at 63.5254 155.0924 0)
-      (effects (font (size 1.27 1.27)) (justify bottom) hide)
-    )
-    (pin "1")
-    (pin "2")
-    (pin "3")
-  )
-  (symbol (lib_id "CatBot_JSC:RGEF300_Fuse") (at 53.086 149.86 0) (unit 1)
+    (property "PARTREV" "C" (id 4) (at 61.722 159.004 0)
+      (effects (font (size 1.27 1.27)) (justify bottom) hide)
+    )
+    (property "STANDARD" "Manufacturer Recommendations" (id 5) (at 72.644 164.338 0)
+      (effects (font (size 1.27 1.27)) (justify bottom) hide)
+    )
+    (property "MAXIMUM_PACKAGE_HEIGHT" "13.59mm" (id 6) (at 70.612 159.004 0)
+      (effects (font (size 1.27 1.27)) (justify bottom) hide)
+    )
+    (property "MANUFACTURER" "E-switch" (id 7) (at 80.518 159.258 0)
+      (effects (font (size 1.27 1.27)) (justify bottom) hide)
+    )
+    (pin "1")
+    (pin "2")
+    (pin "3")
+  )
+  (symbol (lib_id "myKiCadGlobalSymbolLibrary:FUSE") (at 53.086 149.86 0) (unit 1)
     (in_bom yes) (on_board yes)
     (property "Reference" "F1" (id 0) (at 58.166 147.574 0)
@@
       (effects (font (size 1.524 1.524)) hide)
     )
-    (property "Footprint" "myKiCadGlobalFootprintLibrary:RGEF300HF" (id 2) (at 58.166 157.734 0)
+    (property "Footprint" "myKiCadGlobalFootprintLibrary:RGEF300HF" (id 2) (at 58.928 161.036 0)
       (effects (font (size 1.524 1.524)) hide)
     )
@@
     (pin "9")
   )
-  (symbol (lib_id "Power_library:+7.4V") (at 43.688 174.244 0) (unit 1)
+  (symbol (lib_id "myKiCadGlobalSymbolLibrary:+7.4V") (at 43.688 174.244 0) (unit 1)
     (in_bom yes) (on_board yes)
     (property "Reference" "#PWR0101" (id 0) (at 43.688 178.054 0)
@@
     (pin "1")
   )
-  (symbol (lib_id "Molex_connectors_JSC:533750410") (at 268.732 99.06 0) (unit 1)
-    (in_bom yes) (on_board yes)
-    (property "Reference" "J7" (id 0) (at 271.78 92.456 0)
-      (effects (font (size 1.27 1.27)) (justify left))
-    )
-    (property "Value" "533750410" (id 1) (at 277.622 100.3299 0)
-      (effects (font (size 1.27 1.27)) (justify left) hide)
-    )
-    (property "Footprint" "Molex_connectors_JSC:MOLEX_533750410" (id 2) (at 277.622 102.8699 0)
-      (effects (font (size 1.27 1.27)) (justify left) hide)
+  (symbol (lib_id "myKiCadGlobalSymbolLibrary:533750410") (at 268.732 99.06 0) (unit 1)
+    (in_bom yes) (on_board yes)
+    (property "Reference" "J1" (id 0) (at 271.272 92.71 0)
+      (effects (font (size 1.27 1.27)) (justify left bottom))
+    )
+    (property "Value" "533750410" (id 1) (at 268.224 111.76 0)
+      (effects (font (size 1.27 1.27)) (justify left bottom) hide)
+    )
+    (property "Footprint" "myKiCadGlobalFootprintLibrary:533750410" (id 2) (at 270.256 124.46 0)
+      (effects (font (size 1.27 1.27)) (justify bottom) hide)
     )
     (property "Datasheet" "" (id 3) (at 268.732 99.06 0)
       (effects (font (size 1.27 1.27)) hide)
     )
-    (property "PARTREV" "C" (id 4) (at 268.732 99.06 0)
-      (effects (font (size 1.27 1.27)) (justify bottom) hide)
-    )
-    (property "STANDARD" "Manufacturer Recommendations" (id 5) (at 268.224 111.76 0)
-      (effects (font (size 1.27 1.27)) (justify bottom) hide)
-    )
-    (property "MAXIMUM_PACKAGE_HEIGHT" "11.75 mm" (id 6) (at 269.24 113.538 0)
-      (effects (font (size 1.27 1.27)) (justify bottom) hide)
-    )
-    (property "MANUFACTURER" "Molex" (id 7) (at 284.988 113.792 0)
-      (effects (font (size 1.27 1.27)) (justify bottom) hide)
-    )
-    (pin "1")
-    (pin "2")
-    (pin "3")
-    (pin "4")
-  )
-  (symbol (lib_id "Molex_connectors_JSC:0525591853") (at 26.162 29.464 0) (mirror y) (unit 1)
+    (property "PARTREV" "C" (id 4) (at 281.686 123.952 0)
+      (effects (font (size 1.27 1.27)) (justify bottom) hide)
+    )
+    (property "STANDARD" "Manufacturer Recommendations" (id 5) (at 273.05 117.602 0)
+      (effects (font (size 1.27 1.27)) (justify bottom) hide)
+    )
+    (property "MAXIMUM_PACKAGE_HEIGHT" "11.75 mm" (id 6) (at 271.526 121.412 0)
+      (effects (font (size 1.27 1.27)) (justify bottom) hide)
+    )
+    (property "MANUFACTURER" "Molex" (id 7) (at 257.302 124.46 0)
+      (effects (font (size 1.27 1.27)) (justify bottom) hide)
+    )
+    (pin "1")
+    (pin "2")
+    (pin "3")
+    (pin "4")
+  )
+  (symbol (lib_id "myKiCadGlobalSymbolLibrary:525591853") (at 26.162 29.464 0) (mirror y) (unit 1)
     (in_bom yes) (on_board yes) (fields_autoplaced)
     (property "Reference" "J2" (id 0) (at 17.272 24.638 0)
@@
       (effects (font (size 1.524 1.524)) (justify left) hide)
     )
-    (property "Footprint" "Molex_connectors_JSC:CON_525591853_MOL" (id 2) (at 12.7 54.7369 0)
+    (property "Footprint" "myKiCadGlobalFootprintLibrary:525591853" (id 2) (at 12.446 54.7369 0)
       (effects (font (size 1.27 1.27) italic) (justify left) hide)
     )
@@
     (pin "8")
   )
-  (symbol (lib_id "Molex_connectors_JSC:0525591853") (at 262.382 34.036 0) (unit 1)
+  (symbol (lib_id "myKiCadGlobalSymbolLibrary:525591853") (at 262.382 34.036 0) (unit 1)
     (in_bom yes) (on_board yes) (fields_autoplaced)
     (property "Reference" "J9" (id 0) (at 276.606 56.134 0)
@@
       (effects (font (size 1.524 1.524)) (justify left) hide)
     )
-    (property "Footprint" "Molex_connectors_JSC:CON_525591853_MOL" (id 2) (at 276.098 59.3089 0)
+    (property "Footprint" "myKiCadGlobalFootprintLibrary:525591853" (id 2) (at 276.098 59.3089 0)
       (effects (font (size 1.27 1.27) italic) (justify left) hide)
     )
@@
     (pin "2")
   )
-  (symbol (lib_name "12065C503JAT2A_1") (lib_id "myKiCadGlobalSymbolLibrary:12065C503JAT2A") (at 180.34 149.606 90) (unit 1)
+  (symbol (lib_id "myKiCadGlobalSymbolLibrary:12065C503JAT2A") (at 180.34 149.606 90) (unit 1)
     (in_bom yes) (on_board yes)
     (property "Reference" "C1" (id 0) (at 177.038 149.606 0)
@@
       (reference "H4") (unit 1) (value "MountingHole") (footprint "myKiCadGlobalFootprintLibrary:MountingHole_2.2mm_M2")
     )
+    (path "/719a12b3-c9cb-423a-b427-e97a2ca78d9c"
+      (reference "J1") (unit 1) (value "533750410") (footprint "myKiCadGlobalFootprintLibrary:533750410")
+    )
     (path "/7449cb12-a7dc-45a3-9f86-ab09afa5da9d"
-      (reference "J2") (unit 1) (value "0525591853") (footprint "Molex_connectors_JSC:CON_525591853_MOL")
+      (reference "J2") (unit 1) (value "0525591853") (footprint "myKiCadGlobalFootprintLibrary:525591853")
     )
     (path "/dfe34382-e866-481c-ab9b-e4ea9555ce5d"
@@
       (reference "J5") (unit 1) (value "532580229") (footprint "myKiCadGlobalFootprintLibrary:0532580229")
     )
-    (path "/719a12b3-c9cb-423a-b427-e97a2ca78d9c"
-      (reference "J7") (unit 1) (value "533750410") (footprint "Molex_connectors_JSC:MOLEX_533750410")
-    )
     (path "/88fe3ddf-4208-4062-b706-7df06a2f715a"
-      (reference "J9") (unit 1) (value "0525591853") (footprint "Molex_connectors_JSC:CON_525591853_MOL")
+      (reference "J9") (unit 1) (value "0525591853") (footprint "myKiCadGlobalFootprintLibrary:525591853")
     )
     (path "/f63ec720-72b0-4206-a8e7-610e023cb4c0"
